File: I2C-9685-PWM.sch (EAGLE design)
At the start: 34 parts, among them SW1 A0-A3, SW2 A4-A5

Commit message: RR Tracks on back silk, better ground plane
Parts:
- removed R18: 2K0, SPCoast:R0603-RES
- removed R19, R20: 4k7, SPCoast:R0603-RES
- added R7, R8, R9: 10k, SPCoast:R0603-RES
- C1: value 0.1uF -> 220uF; device SPCoast:CAP0805 -> SPCoast:CAP-POL0810
- C4: value 220uF -> 0.1uF; device SPCoast:CAP-POL0810 -> SPCoast:CAP0805
- R1: value 10k -> 2K0
- R2, R3: value 10k -> 4k7
- SW1: value A0-A3 -> A4-A5
- SW2: value A4-A5 -> A0-A3
- renumbered LED18 to LED1, U$2 to U1
Connections:
- net +9V: now also C3.1; no longer C1.1
- net A0: now also R9.1, SW2.1; no longer R6.1, SW1.1
- net A1: now also R8.1, SW2.2; no longer R5.1, SW1.2
- net A2: now also R7.1, SW2.3; no longer R4.1, SW1.3
- net A3: now also R6.1, SW2.4; no longer R3.1, SW1.4
- net A4: now also R5.1, SW1.1; no longer R2.1, SW2.1
- net A5: now also R4.1, SW1.2; no longer R1.1, SW2.2
- net GND: now also C1.-, C4.2, R1.2, SW2.5, SW2.6; no longer C1.2, C4.-, R18.2, SW1.5, SW1.6
- net N$1: now also R1.1; no longer R18.1
- net N$19: now also R3.1; no longer R19.1
- net N$20: now also R2.1; no longer R20.1
- net P1: now also CON4.2; no longer CON1.2
- net P10: now also CON2.3; no longer CON3.3
- net P11: now also CON2.4; no longer CON3.4
- net P12: now also CON2.5; no longer CON3.5
- net P13: now also CON1.2; no longer CON4.2
- net P14: now also CON1.3; no longer CON4.3
- net P15: now also CON1.4; no longer CON4.4
- net P16: now also CON1.5; no longer CON4.5
- net P2: now also CON4.3; no longer CON1.3
- net P3: now also CON4.4; no longer CON1.4
- net P4: now also CON4.5; no longer CON1.5
- net P5: now also CON3.2; no longer CON2.2
- net P6: now also CON3.3; no longer CON2.3
- net P7: now also CON3.4; no longer CON2.4
- net P8: now also CON3.5; no longer CON2.5
- net P9: now also CON2.2; no longer CON3.2
- net SCL: now also R2.2; no longer R20.2
- net SDA: now also R3.2; no longer R19.2
- net VCC: now also C1.+, C4.1, R7.2, R8.2, R9.2; no longer C3.1, C4.+, R1.2, R2.2, R3.2
Other:
- moved on the sheet: C3, CON1, CON2, CON3, CON4, J1, J2, R1, R2, R3, R4, R5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

Commit message: better spacing on IO4s and heatsinking on 7805
Parts:
- SW1: value A4-A5 -> xx xx A5 A4
- SW2: value A0-A3 -> A3 A2 A1 A0
Changed lines of the file:
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@@
 <part name="FID1" library="SPCoast" deviceset="FIDUCIAL" device=""/>
 <part name="FID2" library="SPCoast" deviceset="FIDUCIAL" device=""/>
-<part name="SW2" library="SPCoast" deviceset="SW_DIP-4" device="" value="A0-A3"/>
-<part name="SW1" library="SPCoast" deviceset="SW_DIP-4" device="" value="A4-A5"/>
+<part name="SW2" library="SPCoast" deviceset="SW_DIP-4" device="" value="A3 A2 A1 A0"/>
+<part name="SW1" library="SPCoast" deviceset="SW_DIP-4" device="" value="xx xx A5 A4"/>
 <part name="V5" library="supply2" deviceset="GND" device=""/>
 <part name="C1" library="SPCoast" deviceset="CAP-POL*" device="0810" value="220uF"/>

Commit message: fixed SPCoast lbr part orientation
Parts:
- R1: value 2K0 -> 4k7
Changed lines of the file:
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@@
 <part name="VR1" library="SPCoast" deviceset="VREG-?-*" device="DPAK" technology="5" value="CJ7805"/>
 <part name="P+1" library="supply1" deviceset="VCC" device=""/>
-<part name="R1" library="SPCoast" deviceset="R*" device="0603-RES" value="2K0"/>
+<part name="R1" library="SPCoast" deviceset="R*" device="0603-RES" value="4k7"/>
 <part name="LED1" library="SPCoast" deviceset="LED*" device="0603-LED" value="G"/>
 <part name="SUPPLY2" library="supply2" deviceset="+9V" device=""/>

Commit message: FID placement & names
Parts:
- renumbered FID1 to FID-UL, FID2 to FID-LR
Changed lines of the file:
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@@
 <part name="V12" library="supply2" deviceset="GND" device=""/>
 <part name="BOARD1" library="SPCoast" deviceset="BOARD" device="80X100-IOB" value="BOARD80X100-IOB"/>
-<part name="FID1" library="SPCoast" deviceset="FIDUCIAL" device=""/>
-<part name="FID2" library="SPCoast" deviceset="FIDUCIAL" device=""/>
+<part name="FID-UL" library="SPCoast" deviceset="FIDUCIAL" device=""/>
+<part name="FID-LR" library="SPCoast" deviceset="FIDUCIAL" device=""/>
 <part name="SW2" library="SPCoast" deviceset="SW_DIP-4" device="" value="A3 A2 A1 A0"/>
 <part name="SW1" library="SPCoast" deviceset="SW_DIP-4" device="" value="xx xx A5 A4"/>
@@
 <instance part="V12" gate="GND" x="48.26" y="160.02" rot="R90"/>
 <instance part="BOARD1" gate="B" x="129.54" y="27.94"/>
-<instance part="FID1" gate="FID1" x="243.84" y="48.26"/>
-<instance part="FID2" gate="FID1" x="243.84" y="55.88"/>
+<instance part="FID-UL" gate="FID1" x="243.84" y="48.26"/>
+<instance part="FID-LR" gate="FID1" x="243.84" y="55.88"/>
 <instance part="SW2" gate="A" x="30.48" y="121.92"/>
 <instance part="SW1" gate="A" x="30.48" y="139.7"/>
